File: Hardware/e_book_reader.sch (EAGLE design)
At the start: 103 parts

Commit message: Fixed issue #4 by placing text on info layer
Other:
- note added: "Microcontroller"
- note removed: "ESP32 C6"
