File: Hardware/open-book.brd (EAGLE design)
At the start: 170.2 x 111.2 mm, 103 parts

Commit message: Another quick fix (Changed 3d wires and PCB extra names)
Parts:
- moved SDC_SDC 1.15 mm to (-79.3, 41.5)
- moved SPIESD_D_6 1.15 mm to (-73.2, 44.8)
- moved SDC_C 1.15 mm to (-77.5, 46.5)
- moved SPIESD_R_6 1.15 mm to (-75.9, 46.5)
Routing:
- net GND: track 720.9 -> 724.6 mm, vias 46 -> 48
- net MISO: track 149.1 -> 150.4 mm
- net SS_SD: track 59.8 -> 60.9 mm
- net SCK: track 185.1 -> 186.2 mm
- net MOSI: track 169.3 -> 170.4 mm
- net RESET: track 112.0 -> 112.7 mm
